Commit message: add pick object

File: examples/21-dual_arms_keyboard/panda/panda_arm_with_gripper.urdf (robot description, URDF)
Before this commit: robot panda_arm_with_gripper, 10 links, 9 joints
Links:
- link leftfinger: geometry collision box size=0.04 0.02 0.04; visual box size=0.04 0.02 0.04

Commit message: make sim become more stable

File: examples/21-dual_arms_keyboard/panda/panda_arm_with_gripper.urdf (robot description, URDF)
Before this commit: robot panda_arm_with_gripper, 10 links, 9 joints
Links:
- link leftfinger: geometry collision box size=0.1 0.02 0.1; visual box size=0.1 0.02 0.1
- link rightfinger: geometry collision box size=0.1 0.02 0.1; visual box size=0.1 0.02 0.1

Commit message: enlarge gripper

File: examples/21-dual_arms_keyboard/panda/panda_arm_with_gripper.urdf (robot description, URDF)
Before this commit: robot panda_arm_with_gripper, 10 links, 9 joints
Joints:
- joint finger_joint1: limit lower=0.0 upper=0.04 effort=20 velocity=0.2 -> lower=0.0 upper=0.06 effort=20 velocity=0.2
- joint finger_joint2: limit lower=-0.04 upper=0 effort=20 velocity=0.2 -> lower=-0.06 upper=0 effort=20 velocity=0.2

Commit message: switch key is up

File: examples/21-dual_arms_keyboard/panda/panda_arm_with_gripper.urdf (robot description, URDF)
Before this commit: robot panda_arm_with_gripper, 10 links, 9 joints
Joints:
- joint finger_joint1: limit lower=0.0 upper=0.04 effort=20 velocity=0.2 -> lower=0.0 upper=0.08 effort=200 velocity=1.0
- joint finger_joint2: limit lower=-0.04 upper=0 effort=20 velocity=0.2 -> lower=-0.08 upper=0 effort=200 velocity=1.0
